File: PCB/Alarm clock.kicad_pcb (KiCad board)
At the start: 2 copper layers, 94 x 49 mm, 11 parts, among them J1 Conn_01x08_Pin, SW1 SW_Push, SW2 SW_Push, SW3 SW_Push, SW4 SW_Push, U1 XIAO-ESP32-C3-SMD

Commit message: redid files and actually used git for once
Routing:
- net GND: track 0.00 -> 45.3 mm, vias 0 -> 1
- net Net-(U1-D2): track 27.6 -> 29.9 mm, vias 0 -> 2
